File: Cbil2.kicad_sch (KiCad schematic)
At the start: 26 parts, among them J1 Conn_01x07_Male, U1 430152070826, U2 STM32G030K6T6, U3 HIH7130-000-001, U4 TC72-3.3MUA, U5 KP466PXTMA1, U6 KB_DELPS2.DI-THVG-2J8L-Z555, Y1 ABS07-32.768KHZ-6-4-T

Commit message: Add audio amplifier
Parts:
- removed U2: STM32G030K6T6, symbol sigbo:STM32G030K6T6
- added C12, C13: 10u, symbol Device:C
- added C14, C15: 0.05u, symbol Device:C
- added LS1: Speaker, Buzzer_Beeper:Speaker_CUI_CMR-1206S-67, symbol Device:Speaker
- added R2: 10, symbol Device:R
- added RV1: 10k, symbol Device:R_Potentiometer
- added U7: LM386, symbol Amplifier_Audio:LM386
- added U8: STM32G0B1KETxN, Package_QFP:LQFP-32_7x7mm_P0.8mm, symbol MCU_ST_STM32G0:STM32G0B1KETxN
Connections:
- net VDD_3V3 is gone; now on net VDD: U1.1 (COM_1), U1.3 (COM_2)
- net ADC_1: now also U8.7 (PA0)
- net ADC_2: now also U8.8 (PA1)
- net GND: now also LS1.2, R2.2, RV1.3, U7.2 (-), U7.4 (GND), U8.5 (VSS)
- net NRST: now also U8.6 (PF2)
- net OSC_32_1: now also U8.2 (PC14)
- net OSC_32_2: now also U8.3 (PC15)
- net SPI_MISO: now also U8.13 (PA6)
- net SPI_MOSI: now also U8.9 (PA2)
- net SPI_NCK: now also U8.12 (PA5)
- net SPI_NSS: now also U8.11 (PA4)
- net VDD: now also U8.4 (VDD)
- net 5V: now reaches J1.4 (Pin_4)
- net 5V: now also U7.6 (V+)
- new net: C14.1, C15.1, U7.5
- new net: C14.2, R2.1
- new net: C13.1, RV1.1
- new net: C15.2, LS1.1
- new net: C12.1, U7.8 (GAIN)
- new net: C12.2, U7.1 (GAIN)
- new net: RV1.2, U7.3 (+)
Other:
- moved on the sheet: J1

Commit message: ???
Parts:
- added C16: 4.7uF, Capacitor_SMD:C_0603_1608Metric, symbol Device:C
Connections:
- net GND: now also C16.2
- net VDD: now also U8.20 (VDDIO2), C16.1
Other:
- moved on the sheet: C1, C4
