File: Cbil2.kicad_pcb (KiCad board)
At the start: 2 copper layers, 51.7 x 55.8 mm, 34 parts, among them J1 Conn_01x07_Male, U1 430152070826, U2 TCS40DPR,LF, U3 HIH7130-000-001, U4 TC72-3.3MUA, U5 KP466PXTMA1, U6 KB_DELPS2.DI-THVG-2J8L-Z555, U7 LM386, U8 STM32G0B1KETxN, U9 TCS40DPR,LF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

Commit message: Update layout
Parts:
- added Brd1: SSD1306, SSD1306:128x64OLED, F.Cu at (154.2, 115.9)
- added C20: 4.7uF, Capacitor_SMD:C_0603_1608Metric, F.Cu at (137.3, 115.3)
- added R3: 330, Capacitor_SMD:C_0603_1608Metric, F.Cu at (141.7, 147.3)
- added R4: 330, Capacitor_SMD:C_0603_1608Metric, F.Cu at (145.0, 125.2)
- added R5: 330, Capacitor_SMD:C_0603_1608Metric, F.Cu at (161.5, 107.7)
- added R6: 330, Capacitor_SMD:C_0603_1608Metric, F.Cu at (122.9, 108.2)
- added R7: 10k, Resistor_SMD:R_0603_1608Metric_Pad0.98x0.95mm_HandSolder, F.Cu at (161.5, 113.8)
- added R8: 10k, Resistor_SMD:R_0603_1608Metric_Pad0.98x0.95mm_HandSolder, F.Cu at (161.5, 115.3)
- added U10: KB_DELPS2.DI-THVG-2J8L-Z555, Cbil2-lib:KBDELPS2DITHVG2J8LZ555, F.Cu at (144.1, 122.9)
- added U11: KO DELPS1.22-UGVI-24-H3Q4, Cbil2-lib:KBDELPS2DITHVG2J8LZ555, F.Cu at (161.5, 110.6)
- added U12: KO DELPS1.22-UGVI-24-H3Q4, Cbil2-lib:KBDELPS2DITHVG2J8LZ555, F.Cu at (125.9, 108.2)
- moved C7 13.9 mm to (135.8, 115.3)
- moved C3 13.3 mm to (145.0, 142.2), turned to 90 degrees
- moved R1 2.16 mm to (137.4, 138.9), turned to 180 degrees
Connections:
- J1 pad 4: unconnected-(J1-Pin_4-Pad4) -> /NRST
- J1 pad 5: unconnected-(J1-Pin_5-Pad5) -> /USART_TX
- U1 pad 1: VDD -> GND
- U1 pad 3: VDD -> GND
- U6 pad 2: VDD -> Net-(U6-A)
- U8 pad 1: unconnected-(U8-PB9-Pad1) -> /I2C_SDA
- U8 pad 19: unconnected-(U8-PA9/UCPD1_DBCC1-Pad19) -> /USART_TX
- U8 pad 20: unconnected-(U8-VDDIO2-Pad20) -> VDD
- U8 pad 29: unconnected-(U8-PD3-Pad29) -> /LED
- U8 pad 30: unconnected-(U8-PB6-Pad30) -> /I2C_SCL
Routing:
- net /I2C_SCL: track 0.00 -> 34.4 mm, vias 0 -> 1
- net /I2C_SDA: track 0.00 -> 31.2 mm, vias 0 -> 1
- net VDD: track 133.0 -> 162.7 mm, vias 0 -> 2
- net /USART_TX: track 0.00 -> 26.4 mm, vias 0 -> 2
- net /NRST: track 33.4 -> 51.3 mm
- net GND: track 54.9 -> 69.7 mm, vias 21 -> 26
- net 5V: track 16.7 -> 24.3 mm
- net /DAC_OUT: track 14.9 -> 18.6 mm
- net /LED: track 0.00 -> 3.30 mm
- net Net-(U6-A): track 0.00 -> 2.82 mm
- net Net-(U10-K): track 0.00 -> 2.64 mm
- net Net-(U12-K): track 0.00 -> 2.61 mm
- net Net-(U11-K): track 0.00 -> 2.61 mm
- net /SPI_NSS: track 60.9 -> 58.5 mm
- net /SPI_MISO: track 62.9 -> 61.6 mm
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
Commit message: Add silkscreen
Parts:
- added REF**: KiCad-Logo2_12mm_SilkScreen, Symbol:KiCad-Logo2_12mm_SilkScreen, B.Cu at (143.0, 141.5)
Other:
- board text added: "3V3"
- board text added: "5V"
- board text added: "Al"
- board text added: "CLK"
- board text added: "Cbil2"
- board text added: "GND"
- board text added: "IO"
- board text added: "LED"
- board text added: "Power 3v3"
- board text added: "Power 5V"
- board text added: "RST"
- board text added: "SCL"
- board text added: "SDA"
- board text added: "TX"
- board text added: "v1"
